File: ELECTRICO/frontend_arinc429_lab/frontend_arinc429_tl082_circuit.kicad_sch (KiCad schematic)
At the start: 0 parts

Commit message: electrico: ajusta frontend a componentes adquiridos
Other:
- note added: "1k"
- note added: "22k"
- note added: "33k"
- note added: "38k"
- note added: "6k7"
- note added: "99k"
- note added: "R25"
- note removed: "100k"
- note removed: "20k"
- note removed: "30k"
- note removed: "5k6"
Changed lines of the file:
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@@
 	(title_block
 		(title "Front-end TL082CP ARINC 429-like")
-		(date "2026-07-30")
-		(rev "D")
+		(date "2026-08-05")
+		(rev "E")
 		(company "Proyecto PAMPA")
 	)
@@
 		)
 	)
-	(text "20k"
+	(text "22k"
 		(exclude_from_sim no)
 		(at 81.00 65.00 0)
@@
 		)
 	)
-	(text "30k"
+	(text "33k"
 		(exclude_from_sim no)
 		(at 101.30 51.80 0)
@@
 		)
 	)
-	(text "20k"
+	(text "22k"
 		(exclude_from_sim no)
 		(at 81.00 85.00 0)
@@
 		)
 	)
-	(text "30k"
+	(text "33k"
 		(exclude_from_sim no)
 		(at 101.30 94.80 0)
@@
 		)
 	)
-	(text "20k"
+	(text "22k"
 		(exclude_from_sim no)
 		(at 81.00 160.00 0)
@@
 		)
 	)
-	(text "30k"
+	(text "33k"
 		(exclude_from_sim no)
 		(at 101.30 146.80 0)
@@
 		)
 	)
-	(text "20k"
+	(text "22k"
 		(exclude_from_sim no)
 		(at 81.00 180.00 0)
@@
 		)
 	)
-	(text "30k"
+	(text "33k"
 		(exclude_from_sim no)
 		(at 101.30 189.80 0)
@@
 		)
 	)
-	(text "10k"
+	(text "1k"
 		(exclude_from_sim no)
 		(at 408.30 112.80 0)
@@
 		)
 	)
-	(label "VREF_1V65"
+	(label "VREF_RX"
 		(at 425.00 120.00 0)
 		(effects
@@
 		)
 	)
-	(text "10k"
+	(text "1k"
 		(exclude_from_sim no)
 		(at 408.30 134.80 0)
@@
 	(wire
 		(pts
+			(xy 438.00 192.00) (xy 449.00 192.00)
+		)
+		(stroke
+			(width 0.15)
+			(type solid)
+			(color 140 60 180 255)
+		)
+	)
+	(wire
+		(pts
 			(xy 438.00 192.00) (xy 438.00 196.00)
 		)
@@
 		)
 	)
-	(text "5k6"
+	(text "6k7"
 		(exclude_from_sim no)
 		(at 441.30 204.80 0)
@@
 	(wire
 		(pts
-			(xy 438.00 212.00) (xy 458.00 212.00)
+			(xy 449.00 192.00) (xy 449.00 196.00)
+		)
+		(stroke
+			(width 0.15)
+			(type solid)
+			(color 140 60 180 255)
+		)
+	)
+	(wire
+		(pts
+			(xy 446.50 196.00) (xy 446.50 208.00)
+		)
+		(stroke
+			(width 0.15)
+			(type solid)
+			(color 140 60 180 255)
+		)
+	)
+	(wire
+		(pts
+			(xy 446.50 208.00) (xy 451.50 208.00)
+		)
+		(stroke
+			(width 0.15)
+			(type solid)
+			(color 140 60 180 255)
+		)
+	)
+	(wire
+		(pts
+			(xy 451.50 208.00) (xy 451.50 196.00)
+		)
+		(stroke
+			(width 0.15)
+			(type solid)
+			(color 140 60 180 255)
+		)
+	)
+	(wire
+		(pts
+			(xy 451.50 196.00) (xy 446.50 196.00)
+		)
+		(stroke
+			(width 0.15)
+			(type solid)
+			(color 140 60 180 255)
+		)
+	)
+	(wire
+		(pts
+			(xy 449.00 208.00) (xy 449.00 212.00)
+		)
+		(stroke
+			(width 0.15)
+			(type solid)
+			(color 140 60 180 255)
+		)
+	)
+	(text "R25"
+		(exclude_from_sim no)
+		(at 452.30 200.80 0)
+		(effects
+			(font
+				(size 0.75 0.75)
+				(bold yes)
+			)
+			(justify left bottom)
+		)
+	)
+	(text "38k"
+		(exclude_from_sim no)
+		(at 452.30 204.80 0)
+		(effects
+			(font
+				(size 0.72 0.72)
+			)
+			(justify left bottom)
+		)
+	)
+	(wire
+		(pts
+			(xy 438.00 212.00) (xy 466.00 212.00)
 		)
 		(stroke
@@
 		)
 	)
-	(label "VTH_ACTIVE"
-		(at 458.00 212.00 0)
+	(label "VTH_RX"
+		(at 466.00 212.00 0)
 		(effects
 			(font
@@
 	(wire
 		(pts
-			(xy 458.00 212.00) (xy 458.00 222.00)
+			(xy 466.00 212.00) (xy 466.00 222.00)
 		)
 		(stroke
@@
 	(wire
 		(pts
-			(xy 455.50 222.00) (xy 460.50 222.00)
+			(xy 463.50 222.00) (xy 468.50 222.00)
 		)
 		(stroke
@@
 	(wire
 		(pts
-			(xy 455.50 226.00) (xy 460.50 226.00)
+			(xy 463.50 226.00) (xy 468.50 226.00)
 		)
 		(stroke
@@
 	(wire
 		(pts
-			(xy 458.00 226.00) (xy 458.00 236.00)
+			(xy 466.00 226.00) (xy 466.00 236.00)
 		)
 		(stroke
@@
 	(text "C11"
 		(exclude_from_sim no)
-		(at 461.50 222.60 0)
+		(at 469.50 222.60 0)
 		(effects
 			(font
@@
 	(text "100nF"
 		(exclude_from_sim no)
-		(at 461.50 226.40 0)
+		(at 469.50 226.40 0)
 		(effects
 			(font
@@
 	)
 	(junction
+		(at 438.00 192.00)
+		(diameter 0)
+		(color 140 60 180 255)
+	)
+	(junction
+		(at 449.00 192.00)
+		(diameter 0)
+		(color 140 60 180 255)
+	)
+	(junction
 		(at 438.00 212.00)
 		(diameter 0)
 		(color 140 60 180 255)
 	)
+	(junction
+		(at 449.00 212.00)
+		(diameter 0)
+		(color 140 60 180 255)
+	)
 	(wire
 		(pts
-			(xy 438.00 236.00) (xy 458.00 236.00)
+			(xy 438.00 236.00) (xy 466.00 236.00)
 		)
 		(stroke
@@
 	(wire
 		(pts
-			(xy 448.00 236.00) (xy 448.00 238.30)
+			(xy 452.00 236.00) (xy 452.00 238.30)
 		)
 		(stroke
@@
 	(wire
 		(pts
-			(xy 445.00 238.30) (xy 451.00 238.30)
+			(xy 449.00 238.30) (xy 455.00 238.30)
 		)
 		(stroke
@@
 	(wire
 		(pts
-			(xy 446.00 239.70) (xy 450.00 239.70)
+			(xy 450.00 239.70) (xy 454.00 239.70)
 		)
 		(stroke
@@
 	(wire
 		(pts
-			(xy 447.00 241.00) (xy 449.00 241.00)
+			(xy 451.00 241.00) (xy 453.00 241.00)
 		)
 		(stroke
@@
 		)
 	)
-	(text "100k"
+	(text "99k"
 		(exclude_from_sim no)
 		(at 282.00 65.00 0)
@@
 		)
 	)
-	(text "100k"
+	(text "99k"
 		(exclude_from_sim no)
 		(at 282.00 85.00 0)
@@
 		(color 0 120 0 255)
 	)
-	(label "VREF_1V65"
+	(label "VREF_RX"
 		(at 297.00 104.00 0)
 		(effects
@@
 		)
 	)
-	(text "100k"
+	(text "99k"
 		(exclude_from_sim no)
 		(at 282.00 160.00 0)
@@
 		)
 	)
-	(text "100k"
+	(text "99k"
 		(exclude_from_sim no)
 		(at 282.00 180.00 0)
@@
 		(color 0 120 0 255)
 	)
-	(label "VREF_1V65"
+	(label "VREF_RX"
 		(at 297.00 199.00 0)
 		(effects
@@
 		)
 	)
-	(label "RX_A_BIASED"
+	(label "VTH_RX"
 		(at 466.00 60.00 0)
 		(effects
@@
 		)
 	)
-	(label "VTH_ACTIVE"
+	(label "RX_A_BIASED"
 		(at 466.00 80.00 0)
 		(effects
@@
 		)
 	)
-	(label "RX_B_BIASED"
+	(label "VTH_RX"
 		(at 466.00 155.00 0)
 		(effects
@@
 		)
 	)
-	(label "VTH_ACTIVE"
+	(label "RX_B_BIASED"
 		(at 466.00 175.00 0)
 		(effects
